Commit message: Cleaning up Repo / Adding Rtabmap

File: urdf/_d435.gazebo.xacro (robot description, xacro)
@@ -27,6 +27,6 @@
           <horizontal_fov>${69.4*deg_to_rad}</horizontal_fov>
           <image>
-            <width>1280</width>
-            <height>720</height>
+            <width>640</width>
+            <height>480</height>
             <format>RGB_INT8</format>
           </image>
@@ -63,5 +63,5 @@
           </noise>
         </camera>
-        <always_on>1</always_on>
+        <always_on>0</always_on>
         <update_rate>60</update_rate>
         <visualize>0</visualize>
@@ -85,5 +85,5 @@
           </noise>
         </camera>
-        <always_on>1</always_on>
+        <always_on>0</always_on>
         <update_rate>60</update_rate>
         <visualize>0</visualize>
@@ -93,6 +93,6 @@
           <horizontal_fov>${85.2*deg_to_rad}</horizontal_fov>
           <image>
-            <width>1280</width>
-            <height>720</height>
+            <width>640</width>
+            <height>480</height>
           </image>
           <clip>
@@ -107,5 +107,5 @@
         </camera>
         <always_on>1</always_on>
-        <update_rate>60</update_rate>
+        <update_rate>120</update_rate>
         <visualize>0</visualize>
       </sensor>

File: urdf/little_rover.urdf.xacro (robot description, xacro)
@@ -476,5 +476,5 @@
       <pose>0 0 0 0 0 0</pose>
       <visualize>false</visualize>
-      <update_rate>10</update_rate>
+      <update_rate>30</update_rate>
       <ray>
         <scan>
@@ -482,6 +482,6 @@
             <samples>750</samples>
             <resolution>1</resolution>
-            <min_angle>-1.57</min_angle>
-            <max_angle>1.57</max_angle>
+            <min_angle>-3.14159</min_angle>
+            <max_angle>3.14159</max_angle>
           </horizontal>
         </scan>
@@ -1087,7 +1087,22 @@
     </plugin>
 </gazebo>
+<!-- define the camera parent link
+  <joint name="realsense_cam_joint" type="fixed">
+    <parent link="dummy"/>
+    <child link="realsense_cam"/>
+    <origin xyz="-0.032428513 0 0.063169486" rpy="0 0 0"/>
+  </joint>
+<link name="realsense_cam">
+    <visual>
+        <origin xyz="0 0 0 " rpy="0 0 0"/>
+    </visual>
+    <collision>
+        <origin xyz="0 0 0" rpy="0 0 0"/>
+    </collision>
+  </link>-->
 <!--<link name="dummy" />-->
 <xacro:sensor_d435 name="camera" topics_ns="camera" parent="base_link" publish_pointcloud="true">
-  <origin xyz="-0.032428513 0 0.063169486" rpy="0 0 0" />
+  <!--<origin xyz="-0.032428513 0 0.063169486" rpy="0 0 0" />-->
+  <origin xyz="-0.032428513 0 0.05246948" rpy="0 0 0" />
 </xacro:sensor_d435>
 <!-- Left Wheel Transmission Element -->
